File: floppy.sch (EAGLE design)
At the start: 19 parts, among them IC1 ATTINY13-20SU, Q1 BC547

Commit message: Changed to through-hole AVR Shortened antenna to match 96MHz
Parts:
- removed TP1: TPB1,27, testpad:TPB1,27
- IC1: value ATTINY13-20SU -> ATTINY13-20PU; device attiny13:ATTINY13-20SU -> attiny13:ATTINY13-20PU
Connections:
- net DW: no longer TP1.TP
Changed lines of the file:
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@@
 <part name="G1" library="local" deviceset="BK-913" device=""/>
 <part name="LED1" library="led" deviceset="LED" device="5MM"/>
-<part name="IC1" library="attiny13" deviceset="ATTINY13-20*" device="SU"/>
+<part name="IC1" library="attiny13" deviceset="ATTINY13-20*" device="PU" value="ATTINY13-20PU"/>
 <part name="R1" library="rcl" deviceset="R-EU_" device="0207/7" value="22K"/>
 <part name="P+1" library="supply1" deviceset="VCC" device=""/>
@@
 <part name="P+2" library="supply1" deviceset="VCC" device=""/>
 <part name="GND2" library="supply1" deviceset="GND" device=""/>
-<part name="TP1" library="testpad" deviceset="TP" device="B1,27"/>
 </parts>
 <sheets>
@@
 <instance part="P+2" gate="VCC" x="5.08" y="20.32" rot="R90"/>
 <instance part="GND2" gate="1" x="-2.54" y="20.32"/>
-<instance part="TP1" gate="G$1" x="27.94" y="27.94" rot="R180"/>
 </instances>
 <busses>
@@
 <wire x1="15.24" y1="55.88" x2="17.78" y2="55.88" width="0.1524" layer="91"/>
 <pinref part="JP1" gate="A" pin="1"/>
-<wire x1="17.78" y1="55.88" x2="17.78" y2="33.02" width="0.1524" layer="91"/>
-<pinref part="TP1" gate="G$1" pin="TP"/>
-<wire x1="17.78" y1="33.02" x2="17.78" y2="25.4" width="0.1524" layer="91"/>
-<wire x1="27.94" y1="30.48" x2="27.94" y2="33.02" width="0.1524" layer="91"/>
-<wire x1="27.94" y1="33.02" x2="17.78" y2="33.02" width="0.1524" layer="91"/>
-<junction x="17.78" y="33.02"/>
+<wire x1="17.78" y1="55.88" x2="17.78" y2="25.4" width="0.1524" layer="91"/>
 </segment>
 </net>

Commit message: Changed R1 to 4.7K ohm, which gives much louder sound.
Parts:
- R1: value 22K -> 4.7K
Changed lines of the file:
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@@
 <part name="LED1" library="led" deviceset="LED" device="5MM"/>
 <part name="IC1" library="attiny13" deviceset="ATTINY13-20*" device="PU" value="ATTINY13-20PU"/>
-<part name="R1" library="rcl" deviceset="R-EU_" device="0207/7" value="22K"/>
+<part name="R1" library="rcl" deviceset="R-EU_" device="0207/7" value="4.7K"/>
 <part name="P+1" library="supply1" deviceset="VCC" device=""/>
 <part name="GND1" library="supply1" deviceset="GND" device=""/>

Commit message: Now two batteries Added inductor size too and other minor fixes
Parts:
- added G2: BK-913, local:BK-913
- L1: value (none) -> 62nH
- R1: value 4.7K -> 5.6K
Connections:
- new net N$9: G1.V+, G2.V-
- net VCC: now also G2.V+; no longer G1.V+
Changed lines of the file:
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@@
 <part name="C7" library="rcl" deviceset="C-EU" device="025-025X050" value="22nF"/>
 <part name="Q1" library="transistor-npn" deviceset="BC547*" device="" value="BC547"/>
-<part name="L1" library="rcl" deviceset="L-EU" device="0207/7"/>
+<part name="L1" library="rcl" deviceset="L-EU" device="0207/7" value="62nH"/>
 <part name="S1" library="switch" deviceset="TL36PO" device=""/>
 <part name="G1" library="local" deviceset="BK-913" device=""/>
 <part name="LED1" library="led" deviceset="LED" device="5MM"/>
 <part name="IC1" library="attiny13" deviceset="ATTINY13-20*" device="PU" value="ATTINY13-20PU"/>
-<part name="R1" library="rcl" deviceset="R-EU_" device="0207/7" value="4.7K"/>
+<part name="R1" library="rcl" deviceset="R-EU_" device="0207/7" value="5.6K"/>
 <part name="P+1" library="supply1" deviceset="VCC" device=""/>
 <part name="GND1" library="supply1" deviceset="GND" device=""/>
@@
 <part name="P+2" library="supply1" deviceset="VCC" device=""/>
 <part name="GND2" library="supply1" deviceset="GND" device=""/>
+<part name="G2" library="local" deviceset="BK-913" device=""/>
 </parts>
 <sheets>
@@
 <instance part="P+2" gate="VCC" x="5.08" y="20.32" rot="R90"/>
 <instance part="GND2" gate="1" x="-2.54" y="20.32"/>
+<instance part="G2" gate="G$1" x="154.94" y="88.9" rot="R90"/>
 </instances>
 <busses>
@@
 <junction x="134.62" y="106.68"/>
 <wire x1="63.5" y1="106.68" x2="-12.7" y2="106.68" width="0.1524" layer="91"/>
-<pinref part="G1" gate="G$1" pin="V+"/>
-<wire x1="154.94" y1="83.82" x2="154.94" y2="106.68" width="0.1524" layer="91"/>
 <pinref part="C1" gate="G$1" pin="1"/>
 <pinref part="IC1" gate="G$1" pin="VCC"/>
@@
 <wire x1="-12.7" y1="106.68" x2="-12.7" y2="71.12" width="0.1524" layer="91"/>
 <pinref part="P+1" gate="VCC" pin="VCC"/>
+<pinref part="G2" gate="G$1" pin="V+"/>
+<wire x1="154.94" y1="93.98" x2="154.94" y2="106.68" width="0.1524" layer="91"/>
 <junction x="154.94" y="106.68"/>
+<junction x="-12.7" y="71.12"/>
 </segment>
 <segment>
@@
 <pinref part="GND1" gate="1" pin="GND"/>
 <junction x="157.48" y="38.1"/>
+<junction x="-12.7" y="53.34"/>
 </segment>
 <segment>
@@
 </segment>
 </net>
+<net name="N$9" class="0">
+<segment>
+<pinref part="G1" gate="G$1" pin="V+"/>
+<pinref part="G2" gate="G$1" pin="V-"/>
+</segment>
+</net>
